File: MR BUS BOARD.brd (EAGLE design)
At the start: 127 x 29.5 mm, 34 parts, among them X1 Terminal, X2 Terminal

Commit message: Add files via upload
Parts:
- F1, F2, F3: value PTC FUSE -> 1.5A hold PTC; device adafruit:R1206 -> adafruit:1812
- moved F3 1.96 mm to (57.6, 14.7)
- moved F2 1.45 mm to (61.9, 14.7)
- moved C4 1.42 mm to (67.1, 12.9), turned to 180 degrees
- moved F1 1.14 mm to (71.1, 14.7)
- moved C5 1.02 mm to (67.0, 15.3), turned to 0 degrees
Routing:
- net N$6: track 123.7 -> 139.7 mm
- net GND: track 462.4 -> 473.5 mm, vias 2 -> 4
- net N$14: track 139.6 -> 141.9 mm
- net +5V: track 24.9 -> 26.0 mm
- net N$2: track 141.0 -> 139.9 mm
- net -12V: track 24.9 -> 25.8 mm
- net +12V: track 24.9 -> 25.4 mm
Other:
- board text added: "5/6/23 V1.3"
- board text removed: "5/6/23 V1.2"

Commit message: Add files via upload
Parts:
- F1, F3: value 1.5A hold PTC -> 1.1A hold PTC fuse
- F2: value 1.5A hold PTC -> .5A hold PTC fuse
- R1: value 500 -> 1k
- R2: value 500 -> 330
- R3: value 500 -> 1.2k
Changed lines of the file:
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@@
 <drawing>
 <settings>
-<setting alwaysvectorfont="yes"/>
+<setting alwaysvectorfont="no"/>
 <setting verticaltext="up"/>
 </settings>
@@
 <attribute name="POPULARITY" value="10" x="63.5" y="6.604" size="1.778" layer="27" display="off"/>
 </element>
-<element name="R1" library="rcl" library_urn="urn:adsk.eagle:library:334" package="R0805" package3d_urn="urn:adsk.eagle:package:23553/2" value="500" x="49.657" y="19.431" smashed="yes" rot="R90">
+<element name="R1" library="rcl" library_urn="urn:adsk.eagle:library:334" package="R0805" package3d_urn="urn:adsk.eagle:package:23553/2" value="1k" x="49.657" y="19.431" smashed="yes" rot="R90">
 <attribute name="NAME" x="50.546" y="19.939" size="1.27" layer="25" rot="R270"/>
 <attribute name="POPULARITY" value="85" x="49.657" y="19.431" size="1.778" layer="27" rot="R90" display="off"/>
 <attribute name="SPICEPREFIX" value="R" x="49.657" y="19.431" size="1.778" layer="27" rot="R90" display="off"/>
 </element>
-<element name="R2" library="rcl" library_urn="urn:adsk.eagle:library:334" package="R0805" package3d_urn="urn:adsk.eagle:package:23553/2" value="500" x="49.657" y="9.8425" smashed="yes" rot="R90">
-<attribute name="NAME" x="52.7685" y="11.049" size="1.27" layer="25" rot="R180"/>
+<element name="R2" library="rcl" library_urn="urn:adsk.eagle:library:334" package="R0805" package3d_urn="urn:adsk.eagle:package:23553/2" value="330" x="49.657" y="9.8425" smashed="yes" rot="R90">
+<attribute name="NAME" x="50.673" y="10.8585" size="1.27" layer="25" rot="R270"/>
 <attribute name="POPULARITY" value="85" x="49.657" y="9.8425" size="1.778" layer="27" rot="R90" display="off"/>
 <attribute name="SPICEPREFIX" value="R" x="49.657" y="9.8425" size="1.778" layer="27" rot="R90" display="off"/>
 </element>
-<element name="R3" library="rcl" library_urn="urn:adsk.eagle:library:334" package="R0805" package3d_urn="urn:adsk.eagle:package:23553/2" value="500" x="49.657" y="14.351" smashed="yes" rot="R270">
+<element name="R3" library="rcl" library_urn="urn:adsk.eagle:library:334" package="R0805" package3d_urn="urn:adsk.eagle:package:23553/2" value="1.2k" x="49.657" y="14.351" smashed="yes" rot="R270">
 <attribute name="NAME" x="50.673" y="14.859" size="1.27" layer="25" rot="R270"/>
 <attribute name="POPULARITY" value="85" x="49.657" y="14.351" size="1.778" layer="27" rot="R270" display="off"/>
@@
 <attribute name="NAME" x="121.031" y="25.146" size="1.27" layer="25" ratio="10"/>
 </element>
-<element name="F1" library="adafruit" package="1812" value="1.5A hold PTC" x="71.0565" y="14.732" smashed="yes" rot="R90">
+<element name="F1" library="adafruit" package="1812" value="1.1A hold PTC fuse " x="71.0565" y="14.732" smashed="yes" rot="R90">
 <attribute name="NAME" x="73.5965" y="14.1445" size="0.6096" layer="25" rot="R90"/>
 <attribute name="VALUE" x="69.1515" y="12.8745" size="0.6096" layer="27" rot="R90"/>
 </element>
-<element name="F2" library="adafruit" package="1812" value="1.5A hold PTC" x="61.9125" y="14.732" smashed="yes" rot="R90">
+<element name="F2" library="adafruit" package="1812" value=".5A hold PTC fuse" x="61.9125" y="14.732" smashed="yes" rot="R90">
 <attribute name="NAME" x="64.4525" y="14.1445" size="0.6096" layer="25" rot="R90"/>
 <attribute name="VALUE" x="60.0075" y="12.8745" size="0.6096" layer="27" rot="R90"/>
 </element>
-<element name="F3" library="adafruit" package="1812" value="1.5A hold PTC" x="57.5945" y="14.732" smashed="yes" rot="R90">
+<element name="F3" library="adafruit" package="1812" value="1.1A hold PTC fuse" x="57.5945" y="14.732" smashed="yes" rot="R90">
 <attribute name="NAME" x="55.5625" y="14.1445" size="0.6096" layer="25" rot="R90"/>
 <attribute name="VALUE" x="55.6895" y="12.8745" size="0.6096" layer="27" rot="R90"/>
