File: MR BUS BOARD.sch (EAGLE design)
At the start: 33 parts, among them X1 Terminal, X2 Terminal

Commit message: Add files via upload
Parts:
- F1, F2, F3: value PTC FUSE -> 1.5A hold PTC; device adafruit:PTCFUSE-1206 -> adafruit:PTCFUSE-1812

Commit message: Add files via upload
Parts:
- F1, F3: value 1.5A hold PTC -> 1.1A hold PTC fuse
- F2: value 1.5A hold PTC -> .5A hold PTC fuse
- R1: value 500 -> 1k
- R2: value 500 -> 330
- R3: value 500 -> 1.2k
Changed lines of the file:
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@@
 <part name="JP8" library="pinhead+" deviceset="PINHD-2X8" device="SMT" value="header"/>
 <part name="X1" library="con-wago-500" library_urn="urn:adsk.eagle:library:195" deviceset="W237-4" device="" package3d_urn="urn:adsk.eagle:package:10695/1" value="Terminal"/>
-<part name="R1" library="rcl" library_urn="urn:adsk.eagle:library:334" deviceset="R-US_" device="R0805" package3d_urn="urn:adsk.eagle:package:23553/2" value="500"/>
-<part name="R2" library="rcl" library_urn="urn:adsk.eagle:library:334" deviceset="R-US_" device="R0805" package3d_urn="urn:adsk.eagle:package:23553/2" value="500"/>
-<part name="R3" library="rcl" library_urn="urn:adsk.eagle:library:334" deviceset="R-US_" device="R0805" package3d_urn="urn:adsk.eagle:package:23553/2" value="500"/>
+<part name="R1" library="rcl" library_urn="urn:adsk.eagle:library:334" deviceset="R-US_" device="R0805" package3d_urn="urn:adsk.eagle:package:23553/2" value="1k"/>
+<part name="R2" library="rcl" library_urn="urn:adsk.eagle:library:334" deviceset="R-US_" device="R0805" package3d_urn="urn:adsk.eagle:package:23553/2" value="330"/>
+<part name="R3" library="rcl" library_urn="urn:adsk.eagle:library:334" deviceset="R-US_" device="R0805" package3d_urn="urn:adsk.eagle:package:23553/2" value="1.2k"/>
 <part name="C1" library="rcl" library_urn="urn:adsk.eagle:library:334" deviceset="CPOL-US" device="D" package3d_urn="urn:adsk.eagle:package:23424/2" value="47uf"/>
 <part name="C2" library="rcl" library_urn="urn:adsk.eagle:library:334" deviceset="CPOL-US" device="D" package3d_urn="urn:adsk.eagle:package:23424/2" value="47uf"/>
@@
 <part name="JP15" library="pinhead+" deviceset="PINHD-2X8" device="" value="header1"/>
 <part name="JP16" library="pinhead+" deviceset="PINHD-2X8" device="" value="header1"/>
-<part name="F1" library="adafruit" deviceset="PTCFUSE" device="-1812" value="1.5A hold PTC"/>
-<part name="F2" library="adafruit" deviceset="PTCFUSE" device="-1812" value="1.5A hold PTC"/>
-<part name="F3" library="adafruit" deviceset="PTCFUSE" device="-1812" value="1.5A hold PTC"/>
+<part name="F1" library="adafruit" deviceset="PTCFUSE" device="-1812" value="1.1A hold PTC fuse "/>
+<part name="F2" library="adafruit" deviceset="PTCFUSE" device="-1812" value=".5A hold PTC fuse"/>
+<part name="F3" library="adafruit" deviceset="PTCFUSE" device="-1812" value="1.1A hold PTC fuse"/>
 </parts>
 <sheets>
